Commit message: re-organize the project and start testing ACER algorithm for off-policy actor-critic using MPC data

File: urdfs/quadrotor_base.urdf.xacro (robot description, xacro)
@@ -7,5 +7,5 @@
         <link name="base_link">
             <inertial>
-                <mass value="1.25"/>
+                <mass value="1.00"/>
                 <origin xyz="0 0 0"/>
                 <inertia ixx="0.125" ixy="0.0" ixz="0.0" iyy="0.125" iyz="0.0" izz="0.125"/>
@@ -24,5 +24,6 @@
                 <origin xyz="0 0 0" rpy="0 0 0"/>
                 <geometry>
-                    <box size=".8 .8 .25" />
+                    <!--<box size=".8 .8 .25" />-->
+                    <box size=".8 .8 .36" />
                     <!--<mesh>-->
                         <!--<uri>model://quadrotor/meshes/quadrotor_base.dae</uri>-->

Commit message: disable gazebo contact sensor; test ppo1 only with value initialization; value network should not be updated while learning

File: urdfs/quadrotor_base.urdf.xacro (robot description, xacro)
@@ -7,5 +7,6 @@
         <link name="base_link">
             <inertial>
-                <mass value="1.00"/>
+                <!--<mass value="1.00"/>-->
+                <mass value="1.25" />
                 <origin xyz="0 0 0"/>
                 <inertia ixx="0.125" ixy="0.0" ixz="0.0" iyy="0.125" iyz="0.0" izz="0.125"/>
@@ -25,5 +26,5 @@
                 <geometry>
                     <!--<box size=".8 .8 .25" />-->
-                    <box size=".8 .8 .36" />
+                    <box size=".8 .8 .6" />
                     <!--<mesh>-->
                         <!--<uri>model://quadrotor/meshes/quadrotor_base.dae</uri>-->
