Commit message: change quad_base urdf to calibrate laser sensor measurements

File: urdfs/quadrotor.urdf.xacro (robot description, xacro)
@@ -9,5 +9,5 @@
     <!-- Hokuyo UTM-30LX sensor -->
     <xacro:include filename="$(find hector_sensors_description)/urdf/hokuyo_utm30lx.urdf.xacro" />
-    <xacro:hokuyo_utm30lx name="laser0" parent="base_link" ros_topic="scan" update_rate="40" ray_count="1081" min_angle="-90" max_angle="90">
+    <xacro:hokuyo_utm30lx name="laser0" parent="base_link" ros_topic="scan" update_rate="40" ray_count="1081" min_angle="-80" max_angle="80">
       <origin xyz="0.0 0.0 0.15" rpy="-${M_PI} -${M_PI_2} ${M_PI_2}"/>
     </xacro:hokuyo_utm30lx>

File: urdfs/quadrotor_base.urdf.xacro (robot description, xacro)
@@ -26,5 +26,6 @@
                 <geometry>
                     <!--<box size=".8 .8 .25" />-->
-                    <box size=".8 .8 .6" />
+                    <!--<box size=".8 .8 .6" />-->
+                    <box size=".8 .8 .4" />
                     <!--<mesh>-->
                         <!--<uri>model://quadrotor/meshes/quadrotor_base.dae</uri>-->
